File: ethernet_switcher_hw/MCU.kicad_sch (KiCad schematic)
At the start: 34 parts

Commit message: timer works incorrectly. It's clocked from slower source
Parts:
- removed VD2: DSS34, PcbLib:D_SOD-123F, symbol BluePill-MIK32:Диод Шоттки SOD123FL
Connections:
- net GND: now also XP4.19
- net GPIO1_12: now reaches DD2.1 (P1.12)
- net GPIO1_11: now reaches DD2.2 (P1.11)
- net GPIO1_7: now reaches DD2.21 (P1.7)
- net GPIO1_6: now reaches DD2.22 (P1.6)
- net GPIO1_5: now reaches DD2.23 (P1.5)
- net GPIO1_4: now reaches DD2.25 (P1.4)
- net GPIO1_3: now reaches DD2.26 (P1.3)
- net GPIO1_2: now reaches DD2.27 (P1.2)
- net GPIO1_1: now reaches DD2.28 (P1.1)
- net GPIO1_10: now reaches DD2.3 (P1.10)
- net GPIO1_0: now reaches DD2.30 (P1.0)
- net GPIO2_7: now reaches DD2.31 (P2.7)
- net GPIO2_6: now reaches DD2.32 (P2.6)
- net GPIO2_5: now reaches DD2.33 (SPIFI_D3)
- net GPIO2_4: now reaches DD2.34 (SPIFI_D2)
- net GPIO2_3: now reaches DD2.35 (SPIFI_D1)
- net GPIO2_2: now reaches DD2.36 (SPIFI_D0)
- net GPIO2_1: now reaches DD2.37 (SPIFI_CS)
- net GPIO2_0: now reaches DD2.38 (P2.0)
- net GPIO1_9: now reaches DD2.4 (UART1_TXD)
- net SPI_CS: now reaches DD2.54 (SPI0_CS)
- net SPI_CLK: now reaches DD2.56 (SPI0_CLK)
- net MOSI: now reaches DD2.57 (SPI0_MOSI)
- net MISO: now reaches DD2.58 (SPI0_MISO)
- net GPIO1_8: now reaches DD2.7 (UART1_RXD)
- no-connect marks 13 -> 17
