File: ethernet_switcher_hw/switcher.kicad_sch (KiCad schematic)
At the start: 0 parts

Commit message: timer works incorrectly. It's clocked from slower source
Parts:
- added J3, J4, J6: Conn_02x03_Odd_Even, Connector_PinHeader_2.54mm:PinHeader_2x03_P2.54mm_Vertical, symbol Connector_Generic:Conn_02x03_Odd_Even
- added Q1, Q2, Q3, Q4, Q5, Q6: BSS138, Package_TO_SOT_SMD:SOT-23, symbol Transistor_FET:BSS138
- added R17, R19, R21, R3, R5, R7: 10k, R_0603, symbol Device:R
- added R18, R20, R22, R23, R24, R25, R26, R27, R28, R4, R6, R8: 100k, R_0603, symbol Device:R
Connections:
- new net: Q2.1 (G), R5.1, R6.1
- new net: Q4.1 (G), R17.1, R18.1
- new net: Q3.1 (G), R7.1, R8.1
- new net: Q5.1 (G), R19.1, R20.1
- new net: Q1.1 (G), R3.1, R4.1
- new net: Q6.1 (G), R21.1, R22.1
- new net +3.3V: R23.1, R24.2, R25.1, R26.1, R27.1, R28.1
- new net GND: J3.5 (Pin_5), J3.6 (Pin_6), J4.5 (Pin_5), J4.6 (Pin_6), J6.5 (Pin_5), J6.6 (Pin_6), Q1.2 (S), Q2.2 (S), Q3.2 (S), Q4.2 (S), Q5.2 (S), Q6.2 (S), R18.2, R20.2, R22.2, R4.2, R6.2, R8.2
- new net GPIO1_0_rele_0_position_1: R3.2
- new net GPIO1_10_rele_2_position_1_indicator: J6.2 (Pin_2), R27.2
- new net GPIO1_11_rele_2_position_2_indicator: J6.4 (Pin_4), R28.2
- new net GPIO1_1_rele_0_position_2: R5.2
- new net GPIO1_2_rele_1_position_1: R7.2
- new net GPIO1_3_rele_1_position_2: R17.2
- new net GPIO1_4_rele_2_position_1: R19.2
- new net GPIO1_5_rele_2_position_2: R21.2
- new net GPIO1_6_rele_0_position_1_indicator: J3.2 (Pin_2), R23.2
- new net GPIO1_7_rele_0_position_2_indicator: J3.4 (Pin_4), R24.1
- new net GPIO1_8_rele_1_position_1_indicator: J4.2 (Pin_2), R25.2
- new net GPIO1_9_rele_1_position_2_indicator: J4.4 (Pin_4), R26.2
- new net rele_0_position_1: J3.1 (Pin_1), Q1.3 (D)
- new net rele_0_position_2: J3.3 (Pin_3), Q2.3 (D)
- new net rele_1_position_1: J4.1 (Pin_1), Q3.3 (D)
- new net rele_1_position_2: J4.3 (Pin_3), Q4.3 (D)
- new net rele_2_position_1: J6.1 (Pin_1), Q5.3 (D)
- new net rele_2_position_2: J6.3 (Pin_3), Q6.3 (D)
Other:
- note added: "Indicator Terminals"
- note added: "Power Input Terminals"
- note added: "RELE_0"
- note added: "RELE_1"
- note added: "RELE_2"
