File: ethernet_switcher_hw/w5100.kicad_sch (KiCad schematic)
At the start: 0 parts

Commit message: timer works incorrectly. It's clocked from slower source
Parts:
- added C4, C? (x2): 0.1uF, Capacitor_SMD:C_0402_1005Metric, symbol Device:C_Small
- added C? (x9): 0.1uF, symbol Device:C_Small
- added C? (x2): 13pF, Capacitor_SMD:C_0402_1005Metric, symbol Device:C_Small
- added C?: 3.3uF/16v, symbol Device:C_Small
- added C? (x4): 10uF/16v, symbol Device:C_Small
- added C?: 0.01uF, symbol Device:C_Small
- added D? (x6): LED, LED_SMD:LED_0402_1005Metric, symbol Device:LED
- added J?: RJ45, Connector_RJ:RJ45_Hanrun_HR911105A_Horizontal, symbol Connector:RJ45
- added L?: FB_0805, symbol Device:L_Small
- added L? (x2): 1uH/250mA, symbol Device:L_Small
- added R1, R2, R? (x2): 49.9, Resistor_SMD:R_0402_1005Metric, symbol Device:R_Small
- added R?: 1M, Resistor_SMD:R_0402_1005Metric, symbol Device:R_Small
- added R?: 12k, symbol Device:R_Small
- added R?: 300, symbol Device:R_Small
- added R? (x6): 470, Resistor_SMD:R_0402_1005Metric, symbol Device:R_Small
- added R? (x3): 4k7, symbol Device:R_Small
- added U?: W5100, Package_QFP:LQFP-80_10x10mm_P0.4mm, symbol Interface_Ethernet:W5100
- added Y?: 25Mhz, Crystal:Crystal_HC49-U_Vertical, symbol Device:Crystal
Connections:
- new net: R?.1, U?.1 (RSET_BG)
- new net: R?.1, U?.19 (DATA7), U?.20 (DATA6), U?.21 (DATA5), U?.22 (DATA4), U?.23 (DATA3), U?.24 (DATA2), U?.25 (DATA1), U?.26 (DATA0)
- new net: R?.2, U?.31 (SEN)
- new net: R?.1, U?.38 (ADDR14), U?.39 (ADDR13), U?.40 (ADDR12), U?.41 (ADDR11), U?.42 (ADDR10), U?.45 (ADDR9), U?.46 (ADDR8), U?.47 (ADDR7), U?.48 (ADDR6), U?.49 (ADDR5), U?.50 (ADDR4), U?.51 (ADDR3), U?.52 (ADDR2), U?.53 (ADDR1), U?.54 (ADDR0)
- new net: C?.1, R?.2, R?.2
- new net: C?.2, R1.1, R2.1
- new net: R?.1, R?.2
- new net: D?.2 (A), R?.2 (x6)
- new net +3.3V: C4.1, C?.1, C?.1, C?.1, C?.1, C?.1, C?.1, J?.3, J?.6, L?.1, L?.2, R?.1, R?.1, R?.1, R?.1, R?.1, R?.1
- new net 1V8A: C?.1, L?.2, U?.7 (VCC1V8A), U?.74 (VCC1V8A)
- new net 1V8D: C?.1, C?.1, C?.1, C?.1, C?.1, C?.1, C?.1, C?.1, L?.1, U?.11 (1V8_OUT), U?.15 (VCC1V8D), U?.16 (VCC1V8D), U?.33 (VCC1V8D), U?.69 (VCC1V8D)
- new net 3V3A: U?.2 (VCC3V3A)
- new net 3V3D: R?.1, U?.12 (VCC3V3D), U?.18 (VCC3V3D), U?.44 (VCC3V3D)
- new net COL_LED: D?.1 (K), U?.71 (COLLED)
- new net Earth: C4.2, C?.1, C?.2, C?.2, C?.2, C?.2, C?.2, C?.2, C?.2, C?.2, C?.2, C?.2, C?.2, C?.2, C?.2, C?.2, C?.2, C?.2, C?.2, C?.2, L?.1, L?.2, R?.2, R?.2, R?.2, U?.10 (GNDA), U?.13 (GNDD), U?.14 (GNDD), U?.17 (GNDD), U?.32 (GNDD), U?.34 (TEST_MODE3), U?.35 (TEST_MODE2), U?.36 (TEST_MODE1), U?.37 (TEST_MODE0), U?.4 (GNDA), U?.43 (GNDD), U?.63 (OPMODE0), U?.64 (OPMODE1), U?.65 (OPMODE2), U?.68 (GNDD), U?.77 (GNDA)
- new net FDX_LED: D?.1 (K), U?.70 (FDXLED)
- new net LINK_LED: D?.1 (K), U?.66 (LINKLED)
- new net MISO: U?.27 (MISO)
- new net MOSI: U?.28 (MOSI)
- new net RXIN: J?.8, R2.2, U?.6 (RXIN)
- new net RXIP: J?.7, R1.2, U?.5 (RXIP)
- new net RX_LED: D?.1 (K), U?.72 (RXLED)
- new net SCLK: U?.30 (SCLK)
- new net SCS: U?.29 (~{SCS})
- new net SPD_LED: D?.1 (K), U?.67 (SPDLED)
- new net TXON: J?.2, R?.1, U?.9 (TXON)
- new net TXOP: J?.1, R?.1, U?.8 (TXOP)
- new net TX_LED: D?.1 (K), U?.73 (TXLED)
- new net XTLN: C?.1, R?.2, U?.75 (XTLN), Y?.2
- new net XTLP: C?.1, R?.1, U?.76 (XTLP), Y?.1
Other:
- note added: "1.8v Circuit"
- note added: "25Mhz Crystal"
- note added: "3.3v Circuit"
- note added: "RJ45 Port"
- note added: "U/Pin12"
- note added: "U/Pin15"
- note added: "U/Pin16"
- note added: "U/Pin18"
- note added: "U/Pin33"
- note added: "U/Pin44"
- note added: "U/Pin69"
- note added: "U/Pin7"
- note added: "U/Pin74"
- note added: "W5100"
