File: ethernet_switcher_hw/ethernet_switcher_hw.kicad_sch (KiCad schematic)
At the start: 145 parts, among them Q1 AO3422A, Q10 AO3422A, Q11 AO3422A, Q12 AO3422A, Q13 AO3422A, Q14 AO3422A, Q15 AO3422A, Q16 AO3422A, Q17 NPN, Q18 AO3422A, Q19 AO3422A, Q2 AO3422A, Q20 NPN, Q21 NPN, Q22 AO3422A, Q23 AO3422A, Q24 NPN, Q3 AO3422A, Q4 AO3422A, Q5 AO3422A, Q6 AO3422A, Q7 AO3422A, Q8 AO3422A, Q9 AO3422A, X1 Screw_Terminal_01x02

Commit message: adjustments in scheme
Parts:
- added DD2: K7805-2000R3, K7805-2000R3:CONV_R-78B5.0-1.5, symbol K7805-2000R3:R-78B5.0-1.5
- F1: footprint Fuse:Fuse_0603_1608Metric -> Fuse:Fuse_Bourns_MF-SM_7.98x5.44mm
- R1, R10, R11, R12, R13, R14, R15, R16, R17, R18, R19, R2, R20, R21, R22, R23, R24, R25, R26, R27, R28, R29, R3, R30, R31, R32, R33, R34, R35, R36, R37, R38, R39, R4, R42, R5, R50, R51, R52, R6, R63, R64, R65, R66, R7, R70, R71, R72, R73, R74, R75, R76, R77, R78, R8, R9: footprint Resistor_SMD:R_0603_1608Metric -> Resistor_SMD:R_0805_2012Metric
- R40: renamed from R41; footprint Resistor_SMD:R_0603_1608Metric -> Resistor_SMD:R_0805_2012Metric
- R41: renamed from R40; footprint Resistor_SMD:R_0603_1608Metric -> Resistor_SMD:R_0805_2012Metric
- R43: renamed from R49; footprint Resistor_SMD:R_0603_1608Metric -> Resistor_SMD:R_0805_2012Metric
- R44: renamed from R43; footprint Resistor_SMD:R_0603_1608Metric -> Resistor_SMD:R_0805_2012Metric
- R45: renamed from R44; footprint Resistor_SMD:R_0603_1608Metric -> Resistor_SMD:R_0805_2012Metric
- R46: renamed from R45; footprint Resistor_SMD:R_0603_1608Metric -> Resistor_SMD:R_0805_2012Metric
- R47: renamed from R46; footprint Resistor_SMD:R_0603_1608Metric -> Resistor_SMD:R_0805_2012Metric
- R48: renamed from R47; footprint Resistor_SMD:R_0603_1608Metric -> Resistor_SMD:R_0805_2012Metric
- R49: renamed from R48; footprint Resistor_SMD:R_0603_1608Metric -> Resistor_SMD:R_0805_2012Metric
- R53: renamed from R62; footprint Resistor_SMD:R_0603_1608Metric -> Resistor_SMD:R_0805_2012Metric
- R54: renamed from R53; footprint Resistor_SMD:R_0603_1608Metric -> Resistor_SMD:R_0805_2012Metric
- R55: renamed from R54; footprint Resistor_SMD:R_0603_1608Metric -> Resistor_SMD:R_0805_2012Metric
- R56: renamed from R55; footprint Resistor_SMD:R_0603_1608Metric -> Resistor_SMD:R_0805_2012Metric
- R57: renamed from R56; footprint Resistor_SMD:R_0603_1608Metric -> Resistor_SMD:R_0805_2012Metric
- R58: renamed from R57; footprint Resistor_SMD:R_0603_1608Metric -> Resistor_SMD:R_0805_2012Metric
- R59: renamed from R58; footprint Resistor_SMD:R_0603_1608Metric -> Resistor_SMD:R_0805_2012Metric
- R60: renamed from R59; footprint Resistor_SMD:R_0603_1608Metric -> Resistor_SMD:R_0805_2012Metric
- R61: renamed from R60; footprint Resistor_SMD:R_0603_1608Metric -> Resistor_SMD:R_0805_2012Metric
- R62: renamed from R61; footprint Resistor_SMD:R_0603_1608Metric -> Resistor_SMD:R_0805_2012Metric
- R67: renamed from R69; footprint Resistor_SMD:R_0603_1608Metric -> Resistor_SMD:R_0805_2012Metric
- R68: renamed from R67; footprint Resistor_SMD:R_0603_1608Metric -> Resistor_SMD:R_0805_2012Metric
- R69: renamed from R68; footprint Resistor_SMD:R_0603_1608Metric -> Resistor_SMD:R_0805_2012Metric
- renumbered DD2 to DD3, DD3 to DD4, DD4 to DD5, DD5 to DD6, DD6 to DD7, DD7 to DD8, DD8 to DD9
Connections:
- net +5V: now also DD2.3 (+VOUT)
- net GND: now also DD2.2 (GND)
- net at C1.1, D1.1 (K), DD4.1 (VIN)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: now also DD2.1 (+VIN)
Other:
- note added: "Калачев Д.А."
- note added: "Левченко В.П."

Commit message: final version 1.0
Parts:
- added R79: 1k, Resistor_SMD:R_0805_2012Metric, symbol Device:R
Connections:
- net +3.3V: now also R79.1; no longer X2.12 (+3.3V), X2.15 (+3.3V), X2.18 (+3.3V), X2.21 (+3.3V), X2.24 (+3.3V), X2.27 (+3.3V), X2.3 (+3.3V), X2.30 (+3.3V), X2.6 (+3.3V), X2.9 (+3.3V)
- new net +3.3V_t: R79.2, X2.12 (+3.3V), X2.15 (+3.3V), X2.18 (+3.3V), X2.21 (+3.3V), X2.24 (+3.3V), X2.27 (+3.3V), X2.3 (+3.3V), X2.30 (+3.3V), X2.6 (+3.3V), X2.9 (+3.3V)
Other:
- note added: "АО «НПО «Орион»"
- note added: "МГТУ.468349.001"
- note added: "МГТУ.468349.001 Э3"
- note added: "Схема электрическая"
- note added: "принципиальная"
